File: cad/femto-tia-mainboard.brd (EAGLE design)
At the start: 63.5 x 38.1 mm, 44 parts, among them IC1 LMC6001, IC2 OPA827, IC3 OPA140, IC4 LT3032-5, IC5 LT3032-5, J1 0.125_PAD, X1 SIG_OUT

Commit message: More layout, close to done
Parts:
- removed J1: 0.125_PAD, Kramnik's Library:0.125_PAD
- added U$5, U$6: VIA, 4534:VIA
- IC4, IC5: value LT3032-5 -> LT3032
- R1, R2, R5, R6: device rcl-modified-footprints:R0603 -> rcl-modified-footprints:R0805
- U$2: value VIA -> IN+
- U$3: value VIA -> IN-
- U$4: value VIA -> GND
- moved C22 44.5 mm to (44.1, 5.71), turned to 180 degrees
- moved C24 43.1 mm to (33.0, 14.0)
- moved C26 34.2 mm to (29.2, 13.3), turned to 90 degrees
- moved C25 33.6 mm to (32.4, 5.71), turned to 180 degrees
- moved C21 31.0 mm to (38.1, 9.53), turned to 90 degrees
- moved C23 28.2 mm to (29.2, 7.94), turned to 90 degrees
- moved C13 23.5 mm to (14.3, 14.0), turned to 180 degrees
- moved C14 21.3 mm to (18.7, 14.0), turned to 0 degrees
- moved R2 17.0 mm to (11.1, 17.1), turned to 270 degrees
- moved IC3 16.2 mm to (16.5, 9.53)
- moved C12 11.3 mm to (14.3, 5.08), turned to 180 degrees
- moved C4 10.7 mm to (11.1, 21.3), turned to 90 degrees
- moved C10 10.5 mm to (1.91, 7.62)
- moved U$3 9.55 mm to (50.8, 9.53)
- moved C11 9.23 mm to (18.7, 5.08), turned to 0 degrees
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Connections:
- net N$1 renamed BP_12V
- net N$2 renamed BP_5V
- net N$3 renamed BN_5V
- net N$9 renamed BN_12V
- net VOUT_TIA renamed TIA_VOUT
- removed net N$8: J1.1, R4.S
- new net N$1: IC4.5
- new net N$2: IC5.5
- new net TIA_CF: R4.S, U$5.1, U$6.1
- net GND: now also IC4.4_PAD, IC5.4_PAD; no longer IC4.5, IC5.5
- net PP_N12V0_ANALOG: now also IC5.9_PAD
- net PP_NVIN_D: now also IC4.9_PAD
Routing:
- net PP_N12V0_ANALOG: track 0.00 -> 78.7 mm, vias 0 -> 2
- net PP_P12V0_ANALOG: track 0.00 -> 75.2 mm, vias 0 -> 2
- net VOUT_OFFSET_BUF: track 5.73 -> 46.4 mm
- net GND: track 0.00 -> 35.2 mm, vias 0 -> 22
- net VFB_DRIVER_AMP: track 0.00 -> 18.6 mm
- net PP_N5V0_ANALOG_RC: track 0.00 -> 14.4 mm
- net TIA_VOUT: track 12.2 -> 25.9 mm
- net VOUT_DRIVER_AMP: track 0.00 -> 12.3 mm
- net OFFSET_TRIM: track 0.00 -> 12.1 mm
- net PP_P5V0_ANALOG_RC: track 0.00 -> 8.45 mm
- net PP_P5V0_ANALOG: track 0.00 -> 8.29 mm, vias 0 -> 2
- net BN_5V: track 0.00 -> 7.76 mm, vias 0 -> 2
- net BN_12V: track 0.00 -> 6.30 mm, vias 0 -> 2
- net PP_PVIN: track 0.00 -> 3.95 mm
- net PP_NVIN: track 0.00 -> 3.95 mm
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- added copper zone on layer 1, net GND
- added copper zone on layer 1, net PP_N12V0_ANALOG
- added copper zone on layer 1, net PP_N5V0_ANALOG
- added copper zone on layer 1, net PP_NVIN
- added copper zone on layer 16, net PP_NVIN
- added copper zone on layer 1, net PP_NVIN_D
- added copper zone on layer 1, net PP_P12V0_ANALOG
- added copper zone on layer 1, net PP_P5V0_ANALOG
- added copper zone on layer 1, net PP_PVIN
- added copper zone on layer 16, net PP_PVIN
- added copper zone on layer 1, net PP_PVIN_D
- added copper zone on layer 1, net TIA_CF

Commit message: Done with first-pass routing
Parts:
- U$1: value VIA -> RF
- moved R1 1.35 mm to (24.8, 21.3), turned to 0 degrees
Routing:
- net GND: track 35.2 -> 63.3 mm, vias 22 -> 38
- net PP_P12V0_ANALOG: track 75.2 -> 101.2 mm, vias 2 -> 4
- net PP_N5V0_ANALOG: track 0.00 -> 22.8 mm, vias 0 -> 2
- net TIA_CF: track 0.00 -> 14.3 mm
- net PP_N12V0_ANALOG: track 78.7 -> 88.1 mm
- net PP_P5V0_ANALOG: track 8.29 -> 11.0 mm
- net BN_12V: track 6.30 -> 7.76 mm
- net VOUT_OFFSET_BUF: track 46.4 -> 47.4 mm

Commit message: Exported gerbers and sent out first prototype
Parts:
- removed C25, C26: 10n, rcl:C0603
- removed IC5: LT3032, meng:DFN14-4X3DE
- added C17: 10u, rcl:C1206
- added C18: CAP CER 0.1UF 0805 X7R, rcl-modified-footprints:C0805
- added IC100: LMC6001, femto-tia:DIL08
- added R10: 100k, pot:RJ9W
- added R8, R9: RES SMD 100R 0603 1%, rcl-modified-footprints:R0805
- added TP1, TP6, TP7: GND, Kramnik's Library:KEYSTONE_5000_MINIATURE
- added TP2: FRA_CH2, Kramnik's Library:KEYSTONE_5000_MINIATURE
- added TP3: FRA_CH1, Kramnik's Library:KEYSTONE_5000_MINIATURE
- added TP4: FRA_N, Kramnik's Library:KEYSTONE_5000_MINIATURE
- added TP5: FRA_P, Kramnik's Library:KEYSTONE_5000_MINIATURE
- added U$7: IN-, 4534:VIA
- C10: value CAP CER 0.1UF 0805 X7R -> 10u; device rcl-modified-footprints:C0805 -> rcl:C1206
- C13: value CAP CER 10NF 0805 X7R -> 10u; device rcl-modified-footprints:C0805 -> rcl:C1206
- C14: value CAP CER 0.1UF 0805 X7R -> 10n; device rcl-modified-footprints:C0805 -> rcl:C0603
- C16, C21: value 10u -> 10n; device rcl:C1206 -> rcl:C0603
- C19: value 10n -> 10u; device rcl:C0603 -> rcl:C1206
- C23: value 10u -> CAP CER 0.1UF 0805 X7R; device rcl:C1206 -> rcl-modified-footprints:C0805
- C24: value 10u -> CAP CER 10NF 0805 X7R; device rcl:C1206 -> rcl-modified-footprints:C0805
- C4: value CAP CER 0.1UF 0805 X7R -> (none)
- C5, C7: value CAP CER 10NF 0805 X7R -> CAP CER 0.1UF 0805 X7R
- C6, C8: value CAP CER 0.1UF 0805 X7R -> CAP CER 10NF 0805 X7R
- C9: value (none) -> CAP CER 0.1UF 0805 X7R
- IC1: value LMC6001 -> OPA827; device femto-tia:DIL08 -> femto-tia:SO08
- IC2: value OPA827 -> LT3032; device femto-tia:SO08 -> meng:DFN14-4X3DE
- R1: value RES SMD 100R 0603 1% -> 100k; device rcl-modified-footprints:R0805 -> pot:RJ9W
- R2: value RES SMD 100R 0603 1% -> RES SMD 49R9 1206 1%; device rcl-modified-footprints:R0805 -> rcl-modified-footprints:R1206
- R3: value RES SMD 49R9 1206 1% -> RES SMD 100R 0603 1%; device rcl-modified-footprints:R1206 -> rcl-modified-footprints:R0805
- R4, R7: value 100k -> RES SMD 100R 0603 1%; device pot:RJ9W -> rcl-modified-footprints:R0805
- U$1: value RF -> VIA
- U$2: value IN+ -> VIA
- U$3: value IN- -> VIA
- U$4: value GND -> RF
- U$5: value VIA -> GND
- U$6: value VIA -> IN+
- moved C10 55.8 mm to (56.8, 17.5), turned to 180 degrees
- moved U$6 45.8 mm to (50.8, 14.6)
- moved R2 45.1 mm to (54.3, 30.2), turned to 0 degrees
- moved U$2 44.9 mm to (8.57, 29.8)
- moved U$3 42.6 mm to (13.3, 29.8)
- moved C4 42.1 mm to (53.0, 25.1)
- moved U$5 35.6 mm to (41.3, 15.9)
- moved C9 30.5 mm to (21.3, 20.3), turned to 270 degrees
- moved IC1 30.3 mm to (41.6, 28.3), flipped to the top, turned to 270 degrees
- moved R5 29.7 mm to (19.1, 25.7), turned to 270 degrees
- moved U$4 29.3 mm to (15.6, 29.8)
- moved C7 28.7 mm to (11.1, 21.3), turned to 90 degrees
- moved C2 25.7 mm to (43.8, 32.7), turned to 0 degrees
- moved C1 23.8 mm to (39.4, 32.7), turned to 180 degrees
- moved R7 22.0 mm to (22.5, 24.4), turned to 0 degrees
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Connections:
- new net N$3: R7.2, TP2.P$1, TP4.P$1
- new net N$4: R4.2, TP3.P$1, TP5.P$1
- new net TIA_RF: IC1.3, R1.E, R4.1, R5.1, U$3.1, U$4.1
- net BN_12V: now also C16.1; no longer C19.1
- net BN_5V: now also C20.1, IC2.11; no longer C25.1, IC5.11
- net BP_12V: now also C21.1; no longer C20.1
- net BP_5V: now also C14.1, IC2.3; no longer C26.1, IC5.3
- net GND: now also C17.2, C18.2, C19.2, IC100.3, IC2.4, IC2.4_PAD, R1.A, TP1.P$1, TP6.P$1, TP7.P$1, U$5.1; no longer C14.2, C16.2, C21.2, IC1.3, IC5.4, IC5.4_PAD, R4.A, U$4.1
- net N$2: now also IC2.5; no longer IC5.5
- net NC_TIA_IN: now also IC100.2; no longer IC1.2
- net OFFSET_TRIM: now also C18.1, R10.S; no longer C10.1, R7.S
- net PP_N12V0_ANALOG: now also C16.2, C23.1, C24.1, C5.1, C6.1, IC1.4, IC2.6, IC2.9, IC2.9_PAD, R10.A; no longer C11.1, C12.1, C19.2, C7.1, C8.1, IC2.4, IC5.6, IC5.9, IC5.9_PAD, R7.A
- net PP_N5V0_ANALOG: now also C17.1, C20.2, IC2.7, R9.2; no longer C23.1, C25.2, IC5.7, R2.2
- net PP_N5V0_ANALOG_RC: now also C7.1, IC100.4, R9.1; no longer C4.1, IC1.4, R2.1
- net PP_NVIN: now also U$7.1; no longer U$3.1
- net PP_NVIN_D: now also C19.1; no longer C16.1
- net PP_P12V0_ANALOG: now also C1.1, C11.1, C12.1, C15.1, C2.1, C21.2, IC1.7, IC2.10, IC2.12, IC2.14, R10.E; no longer C13.1, C14.1, C20.2, C21.1, C5.1, C6.1, IC2.7, IC5.10, IC5.12, IC5.14, R7.E
- net PP_P5V0_ANALOG: now also C13.1, C14.2, IC2.1, R8.2; no longer C24.1, C26.2, IC5.1, R1.2
- net PP_P5V0_ANALOG_RC: now also C8.1, C9.1, IC100.7, R8.1; no longer C1.1, C2.1, IC1.7, R1.1
- net PP_PVIN: now also U$6.1; no longer U$2.1
- net PP_PVIN_D: now also C10.1; no longer C15.1
- net TIA_CF: now also R1.S, U$1.1, U$2.1; no longer R4.S, U$5.1, U$6.1
- net TIA_VOUT: now also IC100.6, R5.2, R7.1; no longer IC1.6, IC2.3, R4.E, U$1.1
- net VFB_DRIVER_AMP: now also IC1.2, R3.1; no longer IC2.2, R5.1
- net VOUT: now also R2.2; no longer R3.2
- net VOUT_DRIVER_AMP: now also IC1.6, R2.1, R3.2; no longer IC2.6, R3.1, R5.2
- net VOUT_OFFSET_BUF: now also C4.1; no longer C9.1
Routing:
- net TIA_RF: track 0.00 -> 32.0 mm
- net TIA_VOUT: track 25.9 -> 6.58 mm
- net N$4: track 0.00 -> 13.9 mm
- net N$3: track 0.00 -> 7.30 mm
- net PP_N12V0_ANALOG: track 88.1 -> 91.7 mm
- net TIA_CF: track 14.3 -> 17.9 mm
- net PP_P12V0_ANALOG: track 101.2 -> 97.8 mm
- net PP_P5V0_ANALOG: track 11.0 -> 8.42 mm
- net VOUT_DRIVER_AMP: track 12.3 -> 9.73 mm
- net VFB_DRIVER_AMP: track 18.6 -> 16.0 mm
- net VOUT: track 6.81 -> 5.22 mm
- net VOUT_OFFSET_BUF: track 47.4 -> 48.7 mm
- net GND: track 63.3 -> 63.9 mm, vias 38 -> 86
Other:
- outline, holes or cut-outs redrawn
- board text added: "COMP"
- board text added: "Femtowatt Prototype"
- board text added: "OFFSET"
- board text removed: "Like FEMTO, but a lot cheaper"
