File: cad/femto-tia-mainboard.sch (EAGLE design)
At the start: 44 parts, among them IC1 LMC6001, IC2 OPA827, IC3 OPA140, IC4 LT3032-5, IC5 LT3032-5, J1 0.125_PAD, X1 SIG_OUT

Commit message: More layout, close to done
Parts:
- removed J1: 0.125_PAD, Kramnik's Library:0.125_PAD
- added U$5, U$6: VIA, 4534:VIA
- IC4, IC5: value LT3032-5 -> LT3032
- R1, R2, R5, R6: device rcl-modified-footprints:R-EU_R0603 -> rcl-modified-footprints:R-EU_R0805
- U$2: value VIA -> IN+
- U$3: value VIA -> IN-
- U$4: value VIA -> GND
Connections:
- net VOUT_TIA renamed TIA_VOUT
- removed net N$3: C25.1, IC5.BN
- removed net N$8: J1.1, R4.S
- removed net N$9: C19.1, IC4.BN
- new net BN_12V: C19.1, IC4.BYPN
- new net BN_5V: C25.1, IC5.BYPN
- new net BP_12V: C20.1, IC4.BYPP
- new net BP_5V: C26.1, IC5.BYPP
- new net TIA_CF: R4.S, U$5.P, U$6.P
- net GND: now also IC4.GND4, IC5.GND4; no longer IC4.GND, IC4.GND@1, IC5.GND, IC5.GND@1
- net N$1: now also IC4.GND5; no longer C20.1, IC4.BP
- net N$2: now also IC5.GND5; no longer C26.1, IC5.BP
- net PP_N12V0_ANALOG: now also IC4.OUTN, IC5.INN6, IC5.INN9; no longer IC4.ON, IC5.IN, IC5.IN@1
- net PP_N5V0_ANALOG: now also IC5.OUTN; no longer IC5.ON
- net PP_NVIN_D: now also IC4.INN6, IC4.INN9; no longer IC4.IN, IC4.IN@1
- net PP_P12V0_ANALOG: now also IC4.OUTP, IC5.!SHDNN, IC5.!SHDNP, IC5.INP; no longer IC4.OP, IC5.!SN, IC5.!SP, IC5.IP
- net PP_P5V0_ANALOG: now also IC5.OUTP; no longer IC5.OP
- net PP_PVIN_D: now also IC4.!SHDNN, IC4.!SHDNP, IC4.INP; no longer IC4.!SN, IC4.!SP, IC4.IP
Other:
- note added: "+/- 12V LDO"
- moved on the sheet: C15, C16, C23, C24, C25, C26, D1, D2

Commit message: Done with first-pass routing
Parts:
- U$1: value VIA -> RF
Changed lines of the file:
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@@
 <part name="R6" library="rcl-modified-footprints" deviceset="R-EU_" device="R0805" package3d_urn="urn:adsk.eagle:package:23553/2" value="RES SMD 100R 0603 1%"/>
 <part name="R7" library="pot" library_urn="urn:adsk.eagle:library:331" deviceset="TRIM_EU-" device="RJ9W" package3d_urn="urn:adsk.eagle:package:22702/1" value="100k"/>
-<part name="U$1" library="4534" deviceset="VIA" device=""/>
+<part name="U$1" library="4534" deviceset="VIA" device="" value="RF"/>
 <part name="IC3" library="femto-tia" deviceset="OPA827" device="" value="OPA140"/>
 <part name="C9" library="rcl-modified-footprints" deviceset="C-EU" device="C0805" package3d_urn="urn:adsk.eagle:package:23617/2"/>

Commit message: Exported gerbers and sent out first prototype
Parts:
- removed C25, C26: 10n, rcl:C-EUC0603
- removed IC5: LT3032, meng:LT3032
- added C17: 10u, rcl:C-EUC1206
- added C18: CAP CER 0.1UF 0805 X7R, rcl-modified-footprints:C-EUC0805
- added IC100: LMC6001, femto-tia:LMC6001
- added R10: 100k, pot:TRIM_EU-RJ9W
- added R8, R9: RES SMD 100R 0603 1%, rcl-modified-footprints:R-EU_R0805
- added TP1, TP6, TP7: GND, Kramnik's Library:KEYSTONE_5000
- added TP2: FRA_CH2, Kramnik's Library:KEYSTONE_5000
- added TP3: FRA_CH1, Kramnik's Library:KEYSTONE_5000
- added TP4: FRA_N, Kramnik's Library:KEYSTONE_5000
- added TP5: FRA_P, Kramnik's Library:KEYSTONE_5000
- added U$7: IN-, 4534:VIA
- C10: value CAP CER 0.1UF 0805 X7R -> 10u; device rcl-modified-footprints:C-EUC0805 -> rcl:C-EUC1206
- C13: value CAP CER 10NF 0805 X7R -> 10u; device rcl-modified-footprints:C-EUC0805 -> rcl:C-EUC1206
- C14: value CAP CER 0.1UF 0805 X7R -> 10n; device rcl-modified-footprints:C-EUC0805 -> rcl:C-EUC0603
- C16, C21: value 10u -> 10n; device rcl:C-EUC1206 -> rcl:C-EUC0603
- C19: value 10n -> 10u; device rcl:C-EUC0603 -> rcl:C-EUC1206
- C23: value 10u -> CAP CER 0.1UF 0805 X7R; device rcl:C-EUC1206 -> rcl-modified-footprints:C-EUC0805
- C24: value 10u -> CAP CER 10NF 0805 X7R; device rcl:C-EUC1206 -> rcl-modified-footprints:C-EUC0805
- C4: value CAP CER 0.1UF 0805 X7R -> (none)
- C5, C7: value CAP CER 10NF 0805 X7R -> CAP CER 0.1UF 0805 X7R
- C6, C8: value CAP CER 0.1UF 0805 X7R -> CAP CER 10NF 0805 X7R
- C9: value (none) -> CAP CER 0.1UF 0805 X7R
- IC1: value LMC6001 -> OPA827; device femto-tia:LMC6001 -> femto-tia:OPA827
- IC2: value OPA827 -> LT3032; device femto-tia:OPA827 -> meng:LT3032
- R1: value RES SMD 100R 0603 1% -> 100k; device rcl-modified-footprints:R-EU_R0805 -> pot:TRIM_EU-RJ9W
- R2: value RES SMD 100R 0603 1% -> RES SMD 49R9 1206 1%; device rcl-modified-footprints:R-EU_R0805 -> rcl-modified-footprints:R-EU_R1206
- R3: value RES SMD 49R9 1206 1% -> RES SMD 100R 0603 1%; device rcl-modified-footprints:R-EU_R1206 -> rcl-modified-footprints:R-EU_R0805
- R4, R7: value 100k -> RES SMD 100R 0603 1%; device pot:TRIM_EU-RJ9W -> rcl-modified-footprints:R-EU_R0805
- U$1: value RF -> VIA
- U$2: value IN+ -> VIA
- U$3: value IN- -> VIA
- U$4: value GND -> RF
- U$5: value VIA -> GND
- U$6: value VIA -> IN+
Connections:
- new net N$3: R7.2, TP2.P$1, TP4.P$1
- new net N$4: R4.2, TP3.P$1, TP5.P$1
- new net TIA_RF: IC1.+IN, R1.E, R4.1, R5.1, U$3.P, U$4.P
- net BN_12V: now also C16.1; no longer C19.1
- net BN_5V: now also C20.1, IC2.BYPN; no longer C25.1, IC5.BYPN
- net BP_12V: now also C21.1; no longer C20.1
- net BP_5V: now also C14.1, IC2.BYPP; no longer C26.1, IC5.BYPP
- net GND: now also C17.2, C18.2, C19.2, IC100.+IN, IC2.GND4, R1.A, TP1.P$1, TP6.P$1, TP7.P$1, U$5.P; no longer C14.2, C16.2, C21.2, IC1.+IN, IC5.GND4, R4.A, U$4.P
- net N$2: now also IC2.GND5; no longer IC5.GND5
- net NC_TIA_IN: now also IC100.-IN; no longer IC1.-IN
- net OFFSET_TRIM: now also C18.1, R10.S; no longer C10.1, R7.S
- net PP_N12V0_ANALOG: now also C16.2, C23.1, C24.1, C5.1, C6.1, IC1.V-, IC2.INN6, IC2.INN9, R10.A; no longer C11.1, C12.1, C19.2, C7.1, C8.1, IC2.V-, IC5.INN6, IC5.INN9, R7.A
- net PP_N5V0_ANALOG: now also C17.1, C20.2, IC2.OUTN, R9.2; no longer C23.1, C25.2, IC5.OUTN, R2.2
- net PP_N5V0_ANALOG_RC: now also C7.1, IC100.V-, R9.1; no longer C4.1, IC1.V-, R2.1
- net PP_NVIN: now also U$7.P; no longer U$3.P
- net PP_NVIN_D: now also C19.1; no longer C16.1
- net PP_P12V0_ANALOG: now also C1.1, C11.1, C12.1, C15.1, C2.1, C21.2, IC1.V+, IC2.!SHDNN, IC2.!SHDNP, IC2.INP, R10.E; no longer C13.1, C14.1, C20.2, C21.1, C5.1, C6.1, IC2.V+, IC5.!SHDNN, IC5.!SHDNP, IC5.INP, R7.E
- net PP_P5V0_ANALOG: now also C13.1, C14.2, IC2.OUTP, R8.2; no longer C24.1, C26.2, IC5.OUTP, R1.2
- net PP_P5V0_ANALOG_RC: now also C8.1, C9.1, IC100.V+, R8.1; no longer C1.1, C2.1, IC1.V+, R1.1
- net PP_PVIN: now also U$6.P; no longer U$2.P
- net PP_PVIN_D: now also C10.1; no longer C15.1
- net TIA_CF: now also R1.S, U$1.P, U$2.P; no longer R4.S, U$5.P, U$6.P
- net TIA_VOUT: now also IC100.OUT, R5.2, R7.1; no longer IC1.OUT, IC2.+IN, R4.E, U$1.P
- net VFB_DRIVER_AMP: now also IC1.-IN, R3.1; no longer IC2.-IN, R5.1
- net VOUT: now also R2.2; no longer R3.2
- net VOUT_DRIVER_AMP: now also IC1.OUT, R2.1, R3.2; no longer IC2.OUT, R3.1, R5.2
- net VOUT_OFFSET_BUF: now also C4.1; no longer C9.1
Other:
- moved on the sheet: C1, C10, C11, C12, C13, C14, C15, C16, C19, C2, C20, C21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
